Commit message: new file:   aion_r1_description/meshes/hokuyo.dae 	modified:   aion_r1_description/urdf/r1_sim.urdf.xacro 	modified:   aion_r1_gazebo/models/r1_sim.gazebo 	modified:   aion_r1_gazebo/worlds/aionr1.world 	modified:   ltvcmpc_controller/launch/mpcc_controller.launch 	modified:   ltvcmpc_controller/launch/rover_gazebo.launch 	modified:   ltvcmpc_controller/scripts/__pycache__/ltv_contouring_mpc.cpython-37.pyc 	modified:   ltvcmpc_controller/scripts/data/optimal_path_unicycle.mat 	new file:   ltvcmpc_controller/scripts/data/std_track_optimal.mat 	new file:   ltvcmpc_controller/scripts/data/std_track_optimalx4.mat 	modified:   ltvcmpc_controller/scripts/mpcc_control_node 	modified:   rover_implementation/launch/rover_config.yaml 	new file:   rover_implementation/scripts/pid_angle_node 	new file:   rover_simulation/plots/17-10-2019, 02:36:44/colormap.png 	new file:   rover_simulation/plots/17-10-2019, 02:36:44/inputs.png 	new file:   rover_simulation/plots/17-10-2019, 02:36:44/mpcc_params.txt 	new file:   rover_simulation/plots/17-10-2019, 02:36:44/states.png 	new file:   rover_simulation/plots/17-10-2019, 02:40:38/colormap.png 	new file:   rover_simulation/plots/17-10-2019, 02:40:38/inputs.png 	new file:   rover_simulation/plots/17-10-2019, 02:40:38/mpcc_params.txt 	new file:   rover_simulation/plots/17-10-2019, 02:40:38/states.png 	new file:   rover_simulation/plots/17-10-2019, 02:42:21/colormap.png 	new file:   rover_simulation/plots/17-10-2019, 02:42:21/inputs.png 	new file:   rover_simulation/plots/17-10-2019, 02:42:21/mpcc_params.txt 	new file:   rover_simulation/plots/17-10-2019, 02:42:21/states.png 	new file:   rover_simulation/plots/17-10-2019, 02:42:56/colormap.png 	new file:   rover_simulation/plots/17-10-2019, 02:42:56/inputs.png 	new file:   rover_simulation/plots/17-10-2019, 02:42:56/mpcc_params.txt 	new file:   rover_simulation/plots/17-10-2019, 02:42:56/states.png 	new file:   rover_simulation/plots/17-10-2019, 02:44:09/colormap.png 	new file:   rover_simulation/plots/17-10-2019, 02:44:09/inputs.png 	new file:   rover_simulation/plots/17-10-2019, 02:44:09/mpcc_params.txt 	new file:   rover_simulation/plots/17-10-2019, 02:44:09/states.png 	new file:   rover_simulation/plots/17-10-2019, 02:44:39/colormap.png 	new file:   rover_simulation/plots/17-10-2019, 02:44:39/inputs.png 	new file:   rover_simulation/plots/17-10-2019, 02:44:39/mpcc_params.txt 	new file:   rover_simulation/plots/17-10-2019, 02:44:39/states.png 	new file:   rover_simulation/plots/17-10-2019, 02:45:09/colormap.png 	new file:   rover_simulation/plots/17-10-2019, 02:45:09/inputs.png 	new file:   rover_simulation/plots/17-10-2019, 02:45:09/mpcc_params.txt 	new file:   rover_simulation/plots/17-10-2019, 02:45:09/states.png 	new file:   rover_simulation/plots/17-10-2019, 02:45:36/colormap.png 	new file:   rover_simulation/plots/17-10-2019, 02:45:36/inputs.png 	new file:   rover_simulation/plots/17-10-2019, 02:45:36/mpcc_params.txt 	new file:   rover_simulation/plots/17-10-2019, 02:45:36/states.png 	new file:   rover_simulation/plots/17-10-2019, 02:46:14/colormap.png 	new file:   rover_simulation/plots/17-10-2019, 02:46:14/inputs.png 	new file:   rover_simulation/plots/17-10-2019, 02:46:14/mpcc_params.txt 	new file:   rover_simulation/plots/17-10-2019, 02:46:14/states.png 	new file:   rover_simulation/plots/17-10-2019, 02:47:09/colormap.png 	new file:   rover_simulation/plots/17-10-2019, 02:47:09/inputs.png 	new file:   rover_simulation/plots/17-10-2019, 02:47:09/mpcc_params.txt 	new file:   rover_simulation/plots/17-10-2019, 02:47:09/states.png 	new file:   rover_simulation/plots/17-10-2019, 02:48:12/colormap.png 	new file:   rover_simulation/plots/17-10-2019, 02:48:12/inputs.png 	new file:   rover_simulation/plots/17-10-2019, 02:48:12/mpcc_params.txt 	new file:   rover_simulation/plots/17-10-2019, 02:48:12/states.png 	new file:   rover_simulation/plots/17-10-2019, 02:49:27/colormap.png 	new file:   rover_simulation/plots/17-10-2019, 02:49:27/inputs.png 	new file:   rover_simulation/plots/17-10-2019, 02:49:27/mpcc_params.txt 	new file:   rover_simulation/plots/17-10-2019, 02:49:27/states.png 	new file:   rover_simulation/plots/17-10-2019, 02:51:21/colormap.png 	new file:   rover_simulation/plots/17-10-2019, 02:51:21/inputs.png 	new file:   rover_simulation/plots/17-10-2019, 02:51:21/mpcc_params.txt 	new file:   rover_simulation/plots/17-10-2019, 02:51:21/states.png 	new file:   rover_simulation/plots/17-10-2019, 02:53:13/colormap.png 	new file:   rover_simulation/plots/17-10-2019, 02:53:13/inputs.png 	new file:   rover_simulation/plots/17-10-2019, 02:53:13/mpcc_params.txt 	new file:   rover_simulation/plots/17-10-2019, 02:53:13/states.png 	new file:   rover_simulation/plots/23-10-2019, 16:53:31/colormap.png 	new file:   rover_simulation/plots/23-10-2019, 16:53:31/inputs.png 	new file:   rover_simulation/plots/23-10-2019, 16:53:31/mpcc_params.txt 	new file:   rover_simulation/plots/23-10-2019, 16:53:31/states.png 	new file:   rover_simulation/plots/23-10-2019, 20:47:54/colormap.png 	new file:   rover_simulation/plots/23-10-2019, 20:47:54/inputs.png 	new file:   rover_simulation/plots/23-10-2019, 20:47:54/mpcc_params.txt 	new file:   rover_simulation/plots/23-10-2019, 20:47:54/states.png 	new file:   rover_simulation/plots/23-10-2019, 20:50:41/colormap.png 	new file:   rover_simulation/plots/23-10-2019, 20:50:41/inputs.png 	new file:   rover_simulation/plots/23-10-2019, 20:50:41/mpcc_params.txt 	new file:   rover_simulation/plots/23-10-2019, 20:50:41/states.png 	new file:   rover_simulation/plots/23-10-2019, 20:59:14/colormap.png 	new file:   rover_simulation/plots/23-10-2019, 20:59:14/inputs.png 	new file:   rover_simulation/plots/23-10-2019, 20:59:14/mpcc_params.txt 	new file:   rover_simulation/plots/23-10-2019, 20:59:14/states.png 	new file:   rover_simulation/plots/23-10-2019, 21:02:33/colormap.png 	new file:   rover_simulation/plots/23-10-2019, 21:02:33/inputs.png 	new file:   rover_simulation/plots/23-10-2019, 21:02:33/mpcc_params.txt 	new file:   rover_simulation/plots/23-10-2019, 21:02:33/states.png 	new file:   rover_simulation/plots/23-10-2019, 21:21:43/colormap.png 	new file:   rover_simulation/plots/23-10-2019, 21:21:43/inputs.png 	new file:   rover_simulation/plots/23-10-2019, 21:21:43/mpcc_params.txt 	new file:   rover_simulation/plots/23-10-2019, 21:21:43/states.png 	new file:   rover_simulation/plots/23-10-2019, 22:08:17/colormap.png 	new file:   rover_simulation/plots/23-10-2019, 22:08:17/inputs.png 	new file:   rover_simulation/plots/23-10-2019, 22:08:17/mpcc_params.txt 	new file:   rover_simulation/plots/23-10-2019, 22:08:17/states.png

File: aion_r1_description/urdf/r1_sim.urdf.xacro (robot description, xacro)
@@ -114,5 +114,5 @@
       <material name="gray" />
     </visual>
-    <collision>
+    <!--collision>
       <origin
         xyz="0 0 0.15"
@@ -121,5 +121,5 @@
         <box size="0.455 0.426 0.32" />
       </geometry>
-    </collision>
+    </collision-->
   </link>
   <link
@@ -226,4 +226,33 @@
     <child link="housing_link" />
   </joint>
+  <!--joint
+    name="hokuyo_joint"
+    type="fixed">
+    <origin
+      xyz="0.15 0 0.15"
+      rpy="0 0 0" />
+    <parent link="odom"/>
+    <child link="hokuyo"/>
+  </joint-->
+  <!-- Hokuyo Laser -->
+  <!--link name="hokuyo">
+    <collision>
+      <origin xyz="0 0 0" rpy="0 0 0"/>
+      <geometry>
+    <box size="0.1 0.1 0.1"/>
+      </geometry>
+    </collision>
+    <visual>
+      <origin xyz="0 0 0" rpy="0 0 0"/>
+      <geometry>
+        <mesh filename="package://aion_r1_description/meshes/hokuyo.dae"/>
+      </geometry>
+    </visual>
+    <inertial>
+      <mass value="1e-5" />
+      <origin xyz="0 0 0" rpy="0 0 0"/>
+      <inertia ixx="1e-6" ixy="0" ixz="0" iyy="1e-6" iyz="0" izz="1e-6" />
+    </inertial>
+  </link-->
   <!-- Building links/joints from macros. -->
   <xacro:antenna prefix="l" />
